Commit message: modification

File: description/example_robot.urdf.xacro (robot description, xacro)
@@ -40,5 +40,5 @@
         <child link="link_1"/>
         <axis xyz="0 0 1"/>
-        <limit lower="0" upper="${8*pi/9}" velocity="0.5" effort="100"/>
+        <limit lower="0" upper="5.585" velocity="0.5" effort="100"/>
     </joint>
     <xacro:property name="link_1_length" value="${0.59817}" />
@@ -63,8 +63,8 @@
     </link>
     <!-- Add properties for shoulder -->
-    <xacro:property name="shoulder_length" value="${0.1686 + 0.07493}" />
+    <xacro:property name="shoulder_length" value="${0.1686 + link_1_radius}" />
     <xacro:property name="shoulder_radius" value="${link_1_radius}" />
     <joint name="joint_1_shoulder" type="fixed">
-        <origin xyz="0 0 ${link_1_length}" rpy="-${pi/2} 0 0"/>
+        <origin xyz="0 0 ${link_1_length + shoulder_radius}" rpy="0 0 0"/>
         <parent link="link_1"/>
         <child link="shoulder"/>
@@ -72,5 +72,5 @@
     <link name="shoulder">
         <visual>
-            <origin xyz="0 0 ${shoulder_length/2 - 0.07493}" rpy="0 0 ${pi/2}"/>
+            <origin xyz="0 ${shoulder_length/2 - shoulder_radius} 0" rpy="${pi/2} 0 0"/>
             <geometry>
                 <cylinder length="${shoulder_length}" radius="${shoulder_radius}" />
@@ -79,5 +79,5 @@
         </visual>
         <collision>
-            <origin xyz="0 ${shoulder_length/2 - 0.07493} 0" rpy="0 0 ${pi/2}"/>
+            <origin xyz="0 ${shoulder_length/2 - shoulder_radius} 0" rpy="0 0 ${pi/2}"/>
             <geometry>
                 <cylinder length="${shoulder_length}" radius="${shoulder_radius}" />
@@ -85,19 +85,19 @@
         </collision>
         <xacro:inertial_cylinder mass="0.5" length="${shoulder_length}" radius="${shoulder_radius}">
-            <origin xyz="0 ${shoulder_length/2 - 0.07493} 0" rpy="0 0 ${pi/2}"/>
+            <origin xyz="0 ${shoulder_length/2 - shoulder_radius} 0" rpy="0 0 ${pi/2}"/>
         </xacro:inertial_cylinder>
     </link>
-    <xacro:property name="link_2_length" value="${0.4318 + 0.22606}" />
+    <xacro:property name="link_2_length" value="${0.735}" />
     <xacro:property name="link_2_radius" value="0.065278" />
     <joint name="joint_2" type="revolute">
-        <origin xyz="0 0 ${shoulder_length}" rpy="-${pi/2} 0 0"/>
+        <origin xyz="0 ${shoulder_length} 0" rpy="0 0 0"/>
         <parent link="shoulder"/>
         <child link="link_2"/>
         <axis xyz="0 -1 0"/>
-        <limit lower="0" upper="${25*pi/36}" velocity="0.5" effort="100"/>
+        <limit lower="-1" upper="3.363" velocity="0.5" effort="100"/>
     </joint>
     <link name="link_2">
         <visual>
-            <origin xyz="${link_2_length/2 - 0.22606} 0 0" rpy="0 ${pi/2} 0"/>
+            <origin xyz="${link_2_length/2 - 0.226} 0 0" rpy="0 ${pi/2} 0"/>
             <geometry>
                 <cylinder length="${link_2_length}" radius="${link_2_radius}" />
@@ -106,5 +106,5 @@
         </visual>
         <collision>
-            <origin xyz="${link_2_length/2 - 0.22606} 0 0" rpy="0 ${pi/2} 0"/>
+            <origin xyz="${link_2_length/2 - 0.226} 0 0" rpy="0 ${pi/2} 0"/>
             <geometry>
                 <cylinder length="${link_2_length}" radius="${link_2_radius}" />
@@ -112,5 +112,5 @@
         </collision>
         <xacro:inertial_cylinder mass="1.0" length="${link_2_length}" radius="${link_2_radius}">
-            <origin xyz="${link_2_length/2 - 0.22606} 0 0" rpy="0 ${pi/2} 0"/>
+            <origin xyz="${link_2_length/2 - 0.226} 0 0" rpy="0 ${pi/2} 0"/>
         </xacro:inertial_cylinder>
     </link>
@@ -118,9 +118,9 @@
     <xacro:property name="link_3_radius" value="0.028702" />
     <joint name="joint_3" type="revolute">
-        <origin xyz="${link_2_length - 0.22606} -${link_2_radius + link_3_radius} 0" rpy="0 0 0"/>
+        <origin xyz="${link_2_length - 0.226 - link_3_radius} -${link_2_radius + link_3_radius} 0" rpy="0 0 0"/>
         <parent link="link_2"/>
         <child link="link_3"/>
         <axis xyz="0 -1 0"/>
-        <limit lower="0" upper="${3*pi/4}" velocity="0.5" effort="100"/>
+        <limit lower="-0.712" upper="4" velocity="0.5" effort="100"/>
     </joint>
     <link name="link_3">

Commit message: folder changes

File: description/example_robot.urdf.xacro (robot description, xacro)
@@ -41,4 +41,5 @@
         <axis xyz="0 0 1"/>
         <limit lower="0" upper="5.585" velocity="0.5" effort="100"/>
+        <dynamics damping="10.0" friction="10.0"/>
     </joint>
     <xacro:property name="link_1_length" value="${0.59817}" />
@@ -96,4 +97,5 @@
         <axis xyz="0 -1 0"/>
         <limit lower="-1" upper="3.363" velocity="0.5" effort="100"/>
+        <dynamics damping="10.0" friction="10.0"/>
     </joint>
     <link name="link_2">
@@ -123,4 +125,5 @@
         <axis xyz="0 -1 0"/>
         <limit lower="-0.712" upper="4" velocity="0.5" effort="100"/>
+        <dynamics damping="10.0" friction="10.0"/>
     </joint>
     <link name="link_3">
