Commit message: code update

File: arm_bot/src/description/gazebo_control.xacro (robot description, xacro)
@@ -4,5 +4,5 @@
     <gazebo>
         <plugin name="joint_state_publisher" filename="libgazebo_ros_joint_state_publisher.so">
-            <update_rate>50</update_rate>
+            <update_rate>100</update_rate>
             <joint_name>joint_1</joint_name>
             <joint_name>joint_2</joint_name>
@@ -13,15 +13,15 @@
     <gazebo reference="joint_1">
         <plugin name="joint_1_controller" filename="libgazebo_ros_joint_pose_trajectory.so">
-            <update_rate>50</update_rate>
+            <update_rate>100</update_rate>
         </plugin>
     </gazebo>
     <gazebo reference="joint_2">
         <plugin name="joint_2_controller" filename="libgazebo_ros_joint_pose_trajectory.so">
-            <update_rate>50</update_rate>
+            <update_rate>100</update_rate>
         </plugin>
     </gazebo>
     <gazebo reference="joint_3">
         <plugin name="joint_3_controller" filename="libgazebo_ros_joint_pose_trajectory.so">
-            <update_rate>50</update_rate>
+            <update_rate>100</update_rate>
         </plugin>
     </gazebo>

File: arm_bot/src/description/inertial_macros.xacro (robot description, xacro)
@@ -14,4 +14,10 @@
     <material name="yellow">
         <color rgba="1 1 0 1"/>
+    </material>
+    <material name="green">
+        <color rgba="0.2 1 0.2 1"/>
+    </material>
+    <material name="purple">
+        <color rgba="1 0 1 1"/>
     </material>
     <!-- Specify some standard inertial calculations https://en.wikipedia.org/wiki/List_of_moments_of_inertia -->

File: arm_bot/src/description/robot_core.xacro (robot description, xacro)
@@ -40,11 +40,11 @@
     <link name="link_1">
         <visual>
-            <origin xyz="0 0 ${link_1_length/2}" rpy="0 0 0"/>
-            <!-- <origin xyz="0 0 0" rpy="0 0 ${pi/2}"/> -->
+            <!-- <origin xyz="0 0 ${link_1_length/2}" rpy="0 0 0"/> -->
+            <origin xyz="0 0 0" rpy="0 0 ${-pi/2}"/>
             <geometry>
-                <cylinder length="${link_1_length}" radius="${link_1_radius}" />
-                 <!-- <mesh filename="package://arm_bot/meshes/puma_link1.stl" scale="0.0254 0.0254 0.0254"/> -->
+                <!-- <cylinder length="${link_1_length}" radius="${link_1_radius}" /> -->
+                 <mesh filename="package://arm_bot/meshes/puma_link1.stl" scale="0.0254 0.0254 0.0254"/>
             </geometry>
-            <material name="blue" />
+            <material name="purple" />
         </visual>
         <collision>
@@ -63,5 +63,5 @@
     <xacro:property name="shoulder_radius" value="${link_1_radius}" />
     <joint name="joint_1" type="revolute">
-        <origin xyz="0 0 ${link_1_length + shoulder_radius}" rpy="0 0 0"/>
+        <origin xyz="0 0 0.671" rpy="0 0 0"/>
         <parent link="link_1"/>
         <child link="shoulder"/>
@@ -73,9 +73,9 @@
     <link name="shoulder">
         <visual>
-            <origin xyz="0 ${shoulder_length/2 - shoulder_radius} 0" rpy="${pi/2} 0 0"/>
-            <!-- <origin xyz="0 -0.09677 0" rpy="${pi/2} 0 ${pi}"/> -->
+            <!-- <origin xyz="0 ${shoulder_length/2 - shoulder_radius} 0" rpy="${pi/2} 0 0"/> -->
+            <origin xyz="0 -0.09677 0" rpy="${pi/2} 0 ${pi}"/>
             <geometry>
-                <cylinder length="${shoulder_length}" radius="${shoulder_radius}" />
-                 <!-- <mesh filename="package://arm_bot/meshes/puma_link2.stl" scale="0.0254 0.0254 0.0254"/> -->
+                <!-- <cylinder length="${shoulder_length}" radius="${shoulder_radius}" /> -->
+                 <mesh filename="package://arm_bot/meshes/puma_link2.stl" scale="0.0254 0.0254 0.0254"/>
             </geometry>
             <material name="blue" />
@@ -105,9 +105,9 @@
     <link name="link_2">
         <visual>
-            <origin xyz="${link_2_length/2} 0 0" rpy="0 ${pi/2} 0"/>
-            <!-- <origin xyz="0 0 0" rpy="${3*pi/2} 0 0"/> -->
+            <!-- <origin xyz="${link_2_length/2} 0 0" rpy="0 ${pi/2} 0"/> -->
+            <origin xyz="0 0 0" rpy="0 0 0"/>
             <geometry>
-                <cylinder length="${link_2_length}" radius="${link_2_radius}" />
-                 <!-- <mesh filename="package://arm_bot/meshes/puma_link3.stl" scale="0.0254 0.0254 0.0254"/> -->
+                <!-- <cylinder length="${link_2_length}" radius="${link_2_radius}" /> -->
+                 <mesh filename="package://arm_bot/meshes/puma_link3.stl" scale="0.0254 0.0254 0.0254"/>
             </geometry>
             <material name="orange" />
@@ -137,9 +137,9 @@
     <link name="link_3">
         <visual>
-            <origin xyz="0 -${link_3_length/2} 0" rpy="${-pi/2} 0 0"/>
-            <!-- <origin xyz="0 ${0.094/2} 0" rpy="${pi/2} -${pi/2} 0"/> -->
+            <!-- <origin xyz="0 -${link_3_length/2} 0" rpy="${-pi/2} 0 0"/> -->
+            <origin xyz="0 0 ${0.094/2}" rpy="0 0 ${-pi/2}"/>
             <geometry>
-                <cylinder length="${link_3_length}" radius="${link_3_radius}" />
-                 <!-- <mesh filename="package://arm_bot/meshes/puma_link4.stl" scale="0.0254 0.0254 0.0254"/> -->
+                <!-- <cylinder length="${link_3_length}" radius="${link_3_radius}" /> -->
+                 <mesh filename="package://arm_bot/meshes/puma_link4.stl" scale="0.0254 0.0254 0.0254"/>
             </geometry>
             <material name="yellow" />
@@ -163,5 +163,5 @@
     </gazebo>
     <gazebo reference="link_1">
-        <material>Gazebo/Blue</material>
+        <material>Gazebo/Purple</material>
         <mu1>0.2</mu1>
         <mu2>0.2</mu2>

Commit message: gazebo fortress migration

File: arm_bot/src/description/gazebo_control.xacro (robot description, xacro)
@@ -1,28 +1,20 @@
 <?xml version="1.0"?>
 <robot xmlns:xacro="http://www.ros.org/wiki/xacro">
-    <!-- Joint State Publisher for reading joint positions -->
+    <!-- Ignition Gazebo Fortress: Joint State Publisher -->
+    <!-- Note: In Ignition Gazebo, joint states are typically published via ros_ign_bridge -->
+    <!-- or through the ign_ros2_control plugin when using ros2_control -->
+    <!-- For standalone joint state publishing without ros2_control,
+         you would use ros_ign_bridge to bridge /world/<world_name>/model/<model_name>/joint_state topic -->
+    <!-- If you need direct Ignition Gazebo plugin for joint states: -->
     <gazebo>
-        <plugin name="joint_state_publisher" filename="libgazebo_ros_joint_state_publisher.so">
-            <update_rate>100</update_rate>
+        <plugin filename="ignition-gazebo-joint-state-publisher-system" name="ignition::gazebo::systems::JointStatePublisher">
             <joint_name>joint_1</joint_name>
             <joint_name>joint_2</joint_name>
             <joint_name>joint_3</joint_name>
-        </plugin>
-    </gazebo>
-    <!-- Individual joint control plugins -->
-    <gazebo reference="joint_1">
-        <plugin name="joint_1_controller" filename="libgazebo_ros_joint_pose_trajectory.so">
             <update_rate>100</update_rate>
         </plugin>
     </gazebo>
-    <gazebo reference="joint_2">
-        <plugin name="joint_2_controller" filename="libgazebo_ros_joint_pose_trajectory.so">
-            <update_rate>100</update_rate>
-        </plugin>
-    </gazebo>
-    <gazebo reference="joint_3">
-        <plugin name="joint_3_controller" filename="libgazebo_ros_joint_pose_trajectory.so">
-            <update_rate>100</update_rate>
-        </plugin>
-    </gazebo>
+    <!-- Note: Individual joint pose trajectory controllers are typically handled
+         through ros2_control in Ignition Gazebo rather than separate plugins.
+         If you need trajectory control, use the ros2_control.xacro configuration instead. -->
 </robot>

File: arm_bot/src/description/inertial_macros.xacro (robot description, xacro)
@@ -52,12 +52,14 @@
     <!-- PUMA 560 Specific Inertia Macros based on Stanford paper -->
     <!-- Link 1: Only rotates around Z-axis -->
+    <!-- Modified for Ignition Gazebo compatibility - requires physically valid inertia -->
     <xacro:macro name="inertial_link1" params="*origin">
         <inertial>
             <xacro:insert_block name="origin"/>
-            <!-- Use tiny mass to satisfy RViz, negligible effect on dynamics -->
-            <mass value="0.001" />
+            <!-- Use small but valid mass for Ignition Gazebo -->
+            <mass value="0.1" />
             <!-- Motor inertia Im1=1.14 + Link inertia I1zz=0.35 -->
-            <inertia ixx="0.001" ixy="0.0" ixz="0.0"
-                    iyy="0.001" iyz="0.0"
+            <!-- Adjusted ixx,iyy to be physically valid (must satisfy triangle inequality) -->
+            <inertia ixx="0.75" ixy="0.0" ixz="0.0"
+                    iyy="0.75" iyz="0.0"
                     izz="1.49" />
         </inertial>
@@ -71,6 +73,7 @@
             <!-- I2 = [I2xx, 0, 0; 0, I2yy, 0; 0, 0, I2zz] -->
             <!-- I2xx=0.130, I2yy=0.524, I2zz=0.539+Im2(4.71)=5.249 -->
-            <inertia ixx="0.130" ixy="0.0" ixz="0.0"
-                    iyy="0.524" iyz="0.0"
+            <!-- Adjusted for physical validity: all principal moments must satisfy triangle inequality -->
+            <inertia ixx="2.5" ixy="0.0" ixz="0.0"
+                    iyy="2.8" iyz="0.0"
                     izz="5.249" />
         </inertial>
@@ -84,6 +87,7 @@
             <!-- I3 = [I3xx, 0, 0; 0, I3yy, 0; 0, 0, I3zz] -->
             <!-- I3xx=0.066, I3yy=0.125, I3zz=0.086+Im3(0.83)=0.916 -->
-            <inertia ixx="0.066" ixy="0.0" ixz="0.0"
-                    iyy="0.125" iyz="0.0"
+            <!-- Adjusted for physical validity -->
+            <inertia ixx="0.5" ixy="0.0" ixz="0.0"
+                    iyy="0.5" iyz="0.0"
                     izz="0.916" />
         </inertial>

File: arm_bot/src/description/robot_core.xacro (robot description, xacro)
@@ -155,7 +155,6 @@
         </xacro:inertial_link3>
     </link>
-    <!-- Gazebo-specific properties for links -->
+    <!-- Gazebo-specific properties for links (Ignition Gazebo Fortress compatible) -->
     <gazebo reference="base_link">
-        <material>Gazebo/Green</material>
         <mu1>0.2</mu1>
         <mu2>0.2</mu2>
@@ -163,5 +162,4 @@
     </gazebo>
     <gazebo reference="link_1">
-        <material>Gazebo/Purple</material>
         <mu1>0.2</mu1>
         <mu2>0.2</mu2>
@@ -169,5 +167,4 @@
     </gazebo>
     <gazebo reference="shoulder">
-        <material>Gazebo/Blue</material>
         <mu1>0.2</mu1>
         <mu2>0.2</mu2>
@@ -175,5 +172,4 @@
     </gazebo>
     <gazebo reference="link_2">
-        <material>Gazebo/Orange</material>
         <mu1>0.2</mu1>
         <mu2>0.2</mu2>
@@ -181,5 +177,4 @@
     </gazebo>
     <gazebo reference="link_3">
-        <material>Gazebo/Yellow</material>
         <mu1>0.2</mu1>
         <mu2>0.2</mu2>

File: arm_bot/src/description/ros2_control.xacro (robot description, xacro)
@@ -2,7 +2,8 @@
 <robot xmlns:xacro="http://www.ros.org/wiki/xacro">
     <xacro:if value="$(arg sim_mode)">
-        <ros2_control name="GazeboSystem" type="system">
+        <ros2_control name="GazeboSimSystem" type="system">
             <hardware>
-                <plugin>gazebo_ros2_control/GazeboSystem</plugin>
+                <!-- Gazebo Sim (gz_ros2_control) plugin for Ignition Fortress -->
+                <plugin>gz_ros2_control/GazeboSimSystem</plugin>
             </hardware>
             <joint name="joint_1">
@@ -26,6 +27,7 @@
         </ros2_control>
     </xacro:if>
+    <!-- Gazebo Sim (Ignition Fortress) ros2_control plugin -->
     <gazebo>
-        <plugin name="gazebo_ros2_control" filename="libgazebo_ros2_control.so">
+        <plugin filename="gz_ros2_control-system" name="gz_ros2_control::GazeboSimROS2ControlPlugin">
             <parameters>$(find arm_bot)/config/my_controllers.yaml</parameters>
             <parameters>$(find arm_bot)/config/gaz_ros2_ctl_use_sim.yaml</parameters>
