Commit message: update

File: arm_bot/src/description/inertial_macros.xacro (robot description, xacro)
@@ -44,3 +44,42 @@
         </inertial>
     </xacro:macro>
+    <!-- PUMA 560 Specific Inertia Macros based on Stanford paper -->
+    <!-- Link 1: Only rotates around Z-axis -->
+    <xacro:macro name="inertial_link1" params="*origin">
+        <inertial>
+            <xacro:insert_block name="origin"/>
+            <!-- Use tiny mass to satisfy RViz, negligible effect on dynamics -->
+            <mass value="0.001" />
+            <!-- Motor inertia Im1=1.14 + Link inertia I1zz=0.35 -->
+            <inertia ixx="0.001" ixy="0.0" ixz="0.0"
+                    iyy="0.001" iyz="0.0"
+                    izz="1.49" />
+        </inertial>
+    </xacro:macro>
+    <!-- Link 2 (Shoulder/Upper Arm): m2=17.4 kg -->
+    <!-- CoG w.r.t. link frame: [0.068, 0.006, -0.016] meters -->
+    <xacro:macro name="inertial_link2" params="*origin">
+        <inertial>
+            <xacro:insert_block name="origin"/>
+            <mass value="17.4" />
+            <!-- I2 = [I2xx, 0, 0; 0, I2yy, 0; 0, 0, I2zz] -->
+            <!-- I2xx=0.130, I2yy=0.524, I2zz=0.539+Im2(4.71)=5.249 -->
+            <inertia ixx="0.130" ixy="0.0" ixz="0.0"
+                    iyy="0.524" iyz="0.0"
+                    izz="5.249" />
+        </inertial>
+    </xacro:macro>
+    <!-- Link 3 (Forearm): m3=4.8 kg -->
+    <!-- CoG w.r.t. link frame: [0.000, -0.143, 0.014] meters -->
+    <xacro:macro name="inertial_link3" params="mass *origin">
+        <inertial>
+            <xacro:insert_block name="origin"/>
+            <mass value="${mass}" />
+            <!-- I3 = [I3xx, 0, 0; 0, I3yy, 0; 0, 0, I3zz] -->
+            <!-- I3xx=0.066, I3yy=0.125, I3zz=0.086+Im3(0.83)=0.916 -->
+            <inertia ixx="0.066" ixy="0.0" ixz="0.0"
+                    iyy="0.125" iyz="0.0"
+                    izz="0.916" />
+        </inertial>
+    </xacro:macro>
 </robot>

File: arm_bot/src/description/robot_core.xacro (robot description, xacro)
@@ -82,7 +82,7 @@
             </geometry>
         </collision>
-        <xacro:inertial_cylinder mass="0.5" length="${shoulder_length}" radius="${shoulder_radius}">
-            <origin xyz="0 ${shoulder_length/2 - shoulder_radius} 0" rpy="0 0 ${pi/2}"/>
-        </xacro:inertial_cylinder>
+        <xacro:inertial_link1>
+            <origin xyz="0 0 0" rpy="0 0 0"/>
+        </xacro:inertial_link1>
     </link>
     <xacro:property name="link_2_length" value="0.432" />
@@ -112,7 +112,7 @@
             </geometry>
         </collision>
-        <xacro:inertial_cylinder mass="1.0" length="${link_2_length}" radius="${link_2_radius}">
-            <origin xyz="${link_2_length/2 - 0.226} 0 0" rpy="0 ${pi/2} 0"/>
-        </xacro:inertial_cylinder>
+        <xacro:inertial_link2>
+            <origin xyz="0.068 0.006 -0.016" rpy="0 0 0"/>
+        </xacro:inertial_link2>
     </link>
     <xacro:property name="link_3_length" value="0.233" />
@@ -142,7 +142,38 @@
             </geometry>
         </collision>
-        <xacro:inertial_cylinder mass="0.5" length="${link_3_length}" radius="${link_3_radius}">
-            <origin xyz="0 0 ${link_3_length/2 - 0.4318}" rpy="0 0 0"/>
-        </xacro:inertial_cylinder>
+        <xacro:inertial_link3 mass="4.8">
+            <origin xyz="0.0 -0.143 0.014" rpy="0 0 0"/>
+        </xacro:inertial_link3>
     </link>
+    <!-- Gazebo-specific properties for links -->
+    <gazebo reference="base_link">
+        <material>Gazebo/Green</material>
+        <mu1>0.2</mu1>
+        <mu2>0.2</mu2>
+        <self_collide>true</self_collide>
+    </gazebo>
+    <gazebo reference="link_1">
+        <material>Gazebo/Blue</material>
+        <mu1>0.2</mu1>
+        <mu2>0.2</mu2>
+        <self_collide>true</self_collide>
+    </gazebo>
+    <gazebo reference="shoulder">
+        <material>Gazebo/Blue</material>
+        <mu1>0.2</mu1>
+        <mu2>0.2</mu2>
+        <self_collide>true</self_collide>
+    </gazebo>
+    <gazebo reference="link_2">
+        <material>Gazebo/Orange</material>
+        <mu1>0.2</mu1>
+        <mu2>0.2</mu2>
+        <self_collide>true</self_collide>
+    </gazebo>
+    <gazebo reference="link_3">
+        <material>Gazebo/Yellow</material>
+        <mu1>0.2</mu1>
+        <mu2>0.2</mu2>
+        <self_collide>true</self_collide>
+    </gazebo>
 </robot>

Commit message: fortress finetuning

File: arm_bot/src/description/inertial_macros.xacro (robot description, xacro)
@@ -51,43 +51,59 @@
     </xacro:macro>
     <!-- PUMA 560 Specific Inertia Macros based on Stanford paper -->
-    <!-- Link 1: Only rotates around Z-axis -->
-    <!-- Modified for Ignition Gazebo compatibility - requires physically valid inertia -->
+    <!--
+        INERTIA TENSOR VALIDITY FOR GAZEBO:
+        For a physically valid inertia tensor, the triangle inequality must hold:
+            Ixx + Iyy >= Izz
+            Ixx + Izz >= Iyy
+            Iyy + Izz >= Ixx
+        The original PUMA 560 values have very small Ixx/Iyy relative to Izz because
+        the motor inertia dominates. To satisfy the triangle inequality with MINIMUM
+        deviation from original dynamics:
+        STRATEGY: Set Ixx = Iyy = Izz/2 (minimum valid values)
+        This preserves the critical Izz (rotational inertia about joint axis) while
+        satisfying physics constraints. The Ixx/Iyy values have minimal effect on
+        dynamics since the joints only rotate about the Z-axis.
+    -->
+    <!-- Link 1 (Shoulder): Only rotates around Z-axis -->
+    <!-- Original: m1≈0, Ixx=0.001, Iyy=0.001, Izz=1.49 (Im1=1.14 + I1zz=0.35) -->
+    <!-- Minimum valid: Ixx = Iyy = Izz/2 = 0.745 -->
     <xacro:macro name="inertial_link1" params="*origin">
         <inertial>
             <xacro:insert_block name="origin"/>
-            <!-- Use small but valid mass for Ignition Gazebo -->
-            <mass value="0.1" />
-            <!-- Motor inertia Im1=1.14 + Link inertia I1zz=0.35 -->
-            <!-- Adjusted ixx,iyy to be physically valid (must satisfy triangle inequality) -->
-            <inertia ixx="0.75" ixy="0.0" ixz="0.0"
-                    iyy="0.75" iyz="0.0"
+            <!-- Small mass (original was ~0, but Gazebo needs non-zero) -->
+            <mass value="0.01" />
+            <!-- Izz preserved exactly, Ixx/Iyy set to minimum valid (Izz/2) -->
+            <inertia ixx="0.745" ixy="0.0" ixz="0.0"
+                    iyy="0.745" iyz="0.0"
                     izz="1.49" />
         </inertial>
     </xacro:macro>
-    <!-- Link 2 (Shoulder/Upper Arm): m2=17.4 kg -->
+    <!-- Link 2 (Upper Arm): m2=17.4 kg -->
+    <!-- Original: Ixx=0.130, Iyy=0.524, Izz=5.249 (I2zz=0.539 + Im2=4.71) -->
     <!-- CoG w.r.t. link frame: [0.068, 0.006, -0.016] meters -->
+    <!-- Minimum valid: Ixx = Iyy = Izz/2 = 2.6245 -->
     <xacro:macro name="inertial_link2" params="*origin">
         <inertial>
             <xacro:insert_block name="origin"/>
             <mass value="17.4" />
-            <!-- I2 = [I2xx, 0, 0; 0, I2yy, 0; 0, 0, I2zz] -->
-            <!-- I2xx=0.130, I2yy=0.524, I2zz=0.539+Im2(4.71)=5.249 -->
-            <!-- Adjusted for physical validity: all principal moments must satisfy triangle inequality -->
-            <inertia ixx="2.5" ixy="0.0" ixz="0.0"
-                    iyy="2.8" iyz="0.0"
+            <!-- Izz preserved exactly (critical for joint 2 dynamics) -->
+            <!-- Ixx/Iyy set to minimum valid values -->
+            <inertia ixx="2.6245" ixy="0.0" ixz="0.0"
+                    iyy="2.6245" iyz="0.0"
                     izz="5.249" />
         </inertial>
     </xacro:macro>
     <!-- Link 3 (Forearm): m3=4.8 kg -->
+    <!-- Original: Ixx=0.066, Iyy=0.125, Izz=0.916 (I3zz=0.086 + Im3=0.83) -->
     <!-- CoG w.r.t. link frame: [0.000, -0.143, 0.014] meters -->
+    <!-- Minimum valid: Ixx = Iyy = Izz/2 = 0.458 -->
     <xacro:macro name="inertial_link3" params="mass *origin">
         <inertial>
             <xacro:insert_block name="origin"/>
             <mass value="${mass}" />
-            <!-- I3 = [I3xx, 0, 0; 0, I3yy, 0; 0, 0, I3zz] -->
-            <!-- I3xx=0.066, I3yy=0.125, I3zz=0.086+Im3(0.83)=0.916 -->
-            <!-- Adjusted for physical validity -->
-            <inertia ixx="0.5" ixy="0.0" ixz="0.0"
-                    iyy="0.5" iyz="0.0"
+            <!-- Izz preserved exactly (critical for joint 3 dynamics) -->
+            <!-- Ixx/Iyy set to minimum valid values -->
+            <inertia ixx="0.458" ixy="0.0" ixz="0.0"
+                    iyy="0.458" iyz="0.0"
                     izz="0.916" />
         </inertial>

File: arm_bot/src/description/ros2_control.xacro (robot description, xacro)
@@ -8,5 +8,8 @@
             </hardware>
             <joint name="joint_1">
-                <command_interface name="effort"/>
+                <command_interface name="effort">
+                    <param name="min">-1000</param>
+                    <param name="max">1000</param>
+                </command_interface>
                 <state_interface name="velocity"/>
                 <state_interface name="position"/>
@@ -14,5 +17,8 @@
             </joint>
             <joint name="joint_2">
-                <command_interface name="effort"/>
+                <command_interface name="effort">
+                    <param name="min">-1000</param>
+                    <param name="max">1000</param>
+                </command_interface>
                 <state_interface name="velocity"/>
                 <state_interface name="position"/>
@@ -20,5 +26,8 @@
             </joint>
             <joint name="joint_3">
-                <command_interface name="effort"/>
+                <command_interface name="effort">
+                    <param name="min">-1000</param>
+                    <param name="max">1000</param>
+                </command_interface>
                 <state_interface name="velocity"/>
                 <state_interface name="position"/>

Commit message: tuning

File: arm_bot/src/description/inertial_macros.xacro (robot description, xacro)
@@ -98,8 +98,8 @@
     <!-- CoG w.r.t. link frame: [0.000, -0.143, 0.014] meters -->
     <!-- Minimum valid: Ixx = Iyy = Izz/2 = 0.458 -->
-    <xacro:macro name="inertial_link3" params="mass *origin">
+    <xacro:macro name="inertial_link3" params="*origin">
         <inertial>
             <xacro:insert_block name="origin"/>
-            <mass value="${mass}" />
+            <mass value="4.8" />
             <!-- Izz preserved exactly (critical for joint 3 dynamics) -->
             <!-- Ixx/Iyy set to minimum valid values -->

File: arm_bot/src/description/robot_core.xacro (robot description, xacro)
@@ -63,5 +63,5 @@
     <xacro:property name="shoulder_radius" value="${link_1_radius}" />
     <joint name="joint_1" type="revolute">
-        <origin xyz="0 0 0.671" rpy="0 0 0"/>
+        <origin xyz="0 0 0.6718" rpy="0 0 0"/>
         <parent link="link_1"/>
         <child link="shoulder"/>
@@ -94,5 +94,5 @@
     <xacro:property name="link_2_radius" value="0.065278" />
     <joint name="joint_2" type="revolute">
-        <origin xyz="0 ${shoulder_length} 0" rpy="${-pi/2} 0 0"/>
+        <origin xyz="0 0.2435 0" rpy="${-pi/2} 0 0"/>
         <parent link="shoulder"/>
         <child link="link_2"/>
@@ -126,5 +126,5 @@
     <xacro:property name="link_3_radius" value="0.028702" />
     <joint name="joint_3" type="revolute">
-        <origin xyz="${link_2_length} 0 -0.094" rpy="0 0 0"/>
+        <origin xyz="0.4318 0 -0.094" rpy="0 0 0"/>
         <parent link="link_2"/>
         <child link="link_3"/>
@@ -151,5 +151,5 @@
             </geometry>
         </collision>
-        <xacro:inertial_link3 mass="4.8">
+        <xacro:inertial_link3>
             <origin xyz="0.0 -0.143 0.014" rpy="0 0 0"/>
         </xacro:inertial_link3>
