Commit message: update

File: arm_bot/src/description/robot_core.xacro (robot description, xacro)
@@ -45,5 +45,6 @@
         <origin xyz="0 0 ${link_1_length/2}" rpy="0 0 0"/>
         <geometry>
-            <cylinder length="${link_1_length}" radius="${link_1_radius}" />
+            <!-- <cylinder length="${link_1_length}" radius="${link_1_radius}" /> -->
+                <mesh filename="package://arm_bot/meshes/base_link.STL" scale="1 1 1"/>
         </geometry>
         <material name="blue" />
@@ -69,12 +70,13 @@
     <link name="shoulder">
         <visual>
-            <origin xyz="0 ${shoulder_length/2 - shoulder_radius} 0" rpy="${pi/2} 0 0"/>
+            <origin xyz="0 ${shoulder_length/2 - shoulder_radius} 0" rpy="0 0 0"/>
             <geometry>
-                <cylinder length="${shoulder_length}" radius="${shoulder_radius}" />
+                <!-- <cylinder length="${shoulder_length}" radius="${shoulder_radius}" /> -->
+                <mesh filename="package://arm_bot/meshes/link_1.STL" scale="1 1 1"/>
             </geometry>
             <material name="blue" />
         </visual>
         <collision>
-            <origin xyz="0 ${shoulder_length/2 - shoulder_radius} 0" rpy="0 0 ${pi/2}"/>
+            <origin xyz="0 ${shoulder_length/2 - shoulder_radius} 0" rpy="0 0 0"/>
             <geometry>
                 <cylinder length="${shoulder_length}" radius="${shoulder_radius}" />
@@ -82,5 +84,5 @@
         </collision>
         <xacro:inertial_cylinder mass="0.5" length="${shoulder_length}" radius="${shoulder_radius}">
-            <origin xyz="0 ${shoulder_length/2 - shoulder_radius} 0" rpy="0 0 ${pi/2}"/>
+            <origin xyz="0 ${shoulder_length/2 - shoulder_radius} 0" rpy="0 0 0"/>
         </xacro:inertial_cylinder>
     </link>
@@ -97,13 +99,13 @@
     <link name="link_2">
         <visual>
-            <origin xyz="${link_2_length/2 - 0.226} 0 0" rpy="${3*pi/2} 0 0"/>
+            <origin xyz="${link_2_length/2 - 0.226} 0 0" rpy="0 0 0"/>
             <geometry>
                 <!-- <cylinder length="${link_2_length}" radius="${link_2_radius}" /> -->
-                <mesh filename="package://arm_bot/meshes/puma_link3.stl" scale="26.15 26.15 26.15"/>
+                <mesh filename="package://arm_bot/meshes/link_2.STL" scale="1 1 1"/>
             </geometry>
             <material name="orange" />
         </visual>
         <collision>
-            <origin xyz="${link_2_length/2 - 0.226} 0 0" rpy="0 ${pi/2} 0"/>
+            <origin xyz="${link_2_length/2 - 0.226} 0 0" rpy="0 0 0"/>
             <geometry>
                 <cylinder length="${link_2_length}" radius="${link_2_radius}" />
@@ -112,5 +114,5 @@
         </collision>
         <xacro:inertial_cylinder mass="1.0" length="${link_2_length}" radius="${link_2_radius}">
-            <origin xyz="${link_2_length/2 - 0.226} 0 0" rpy="0 ${pi/2} 0"/>
+            <origin xyz="${link_2_length/2 - 0.226} 0 0" rpy="0 0 0"/>
         </xacro:inertial_cylinder>
     </link>
@@ -129,5 +131,6 @@
             <origin xyz="0 0 ${link_3_length/2 - 0.4318}" rpy="0 0 0"/>
             <geometry>
-                <cylinder length="${link_3_length}" radius="${link_3_radius}" />
+                <!-- <cylinder length="${link_3_length}" radius="${link_3_radius}" /> -->
+                <mesh filename="package://arm_bot/meshes/link_3.STL" scale="1 1 1"/>
             </geometry>
             <material name="yellow" />

Commit message: model update

File: arm_bot/src/description/robot_core.xacro (robot description, xacro)
@@ -1,4 +1,4 @@
 <?xml version="1.0"?>
-<robot xmlns:xacro="http://www.ros.org/wiki/xacro"  name="robot">
+<robot xmlns:xacro="http://www.ros.org/wiki/xacro" name="robot">
     <xacro:include filename="inertial_macros.xacro" />
     <!-- This first link called "world" is empty -->
@@ -31,40 +31,41 @@
         </inertial>
     </link>
-    <joint name="joint_1" type="revolute">
+    <joint name="joint_1_shoulder" type="fixed">
         <origin xyz="0 0 0.1" rpy="0 0 0"/>
         <parent link="base_link"/>
         <child link="link_1"/>
+    </joint>
+    <xacro:property name="link_1_length" value="0.59817" />
+    <xacro:property name="link_1_radius" value="0.07493" />
+    <link name="link_1">
+        <visual>
+            <origin xyz="0 0 ${link_1_length/2}" rpy="0 0 0"/>
+            <geometry>
+                <cylinder length="${link_1_length}" radius="${link_1_radius}" />
+            </geometry>
+            <material name="blue" />
+        </visual>
+        <collision>
+            <origin xyz="0 0 ${link_1_length/2}" rpy="0 0 0"/>
+            <geometry>
+                <cylinder length="${link_1_length}" radius="${link_1_radius}" />
+            </geometry>
+        </collision>
+        <xacro:inertial_cylinder mass="0.5" length="${link_1_length}" radius="${link_1_radius}">
+            <origin xyz="0 0 ${link_1_length/2}" rpy="0 0 0"/>
+        </xacro:inertial_cylinder>
+    </link>
+    <!-- Add properties for shoulder -->
+    <xacro:property name="shoulder_length" value="${0.1686 + link_1_radius}" />
+    <xacro:property name="shoulder_radius" value="${link_1_radius}" />
+    <joint name="joint_1" type="revolute">
+        <origin xyz="0 0 ${link_1_length + shoulder_radius}" rpy="0 0 0"/>
+        <parent link="link_1"/>
+        <child link="shoulder"/>
         <axis xyz="0 0 1"/>
         <limit lower="0" upper="5.585" velocity="1" effort="100"/>
         <dynamics damping="1.0" friction="1.0"/>
     </joint>
-    <xacro:property name="link_1_length" value="${0.59817}" />
-    <xacro:property name="link_1_radius" value="0.07493" />
-    <link name="link_1">
-    <visual>
-        <origin xyz="0 0 ${link_1_length/2}" rpy="0 0 0"/>
-        <geometry>
-            <cylinder length="${link_1_length}" radius="${link_1_radius}" />
-        </geometry>
-        <material name="blue" />
-    </visual>
-    <collision>
-        <origin xyz="0 0 ${link_1_length/2}" rpy="0 0 0"/>
-        <geometry>
-            <cylinder length="${link_1_length}" radius="${link_1_radius}" />
-        </geometry>
-    </collision>
-    <xacro:inertial_cylinder mass="0.5" length="${link_1_length}" radius="${link_1_radius}">
-        <origin xyz="0 0 ${link_1_length/2}" rpy="0 0 0"/>
-    </xacro:inertial_cylinder>
-    </link>
-    <!-- Add properties for shoulder -->
-    <xacro:property name="shoulder_length" value="${0.1686 + link_1_radius}" />
-    <xacro:property name="shoulder_radius" value="${link_1_radius}" />
-    <joint name="joint_1_shoulder" type="fixed">
-        <origin xyz="0 0 ${link_1_length + shoulder_radius}" rpy="0 0 0"/>
-        <parent link="link_1"/>
-        <child link="shoulder"/>
-    </joint>
+    <!-- MATLAB Link 1 = shoulder (m1=0, only Izz=1.49) -->
     <link name="shoulder">
         <visual>
@@ -76,5 +77,5 @@
         </visual>
         <collision>
-            <origin xyz="0 ${shoulder_length/2 - shoulder_radius} 0" rpy="0 0 ${pi/2}"/>
+            <origin xyz="0 ${shoulder_length/2 - shoulder_radius} 0" rpy="${pi/2} 0 0"/>
             <geometry>
                 <cylinder length="${shoulder_length}" radius="${shoulder_radius}" />
@@ -85,5 +86,5 @@
         </xacro:inertial_cylinder>
     </link>
-    <xacro:property name="link_2_length" value="${0.735}" />
+    <xacro:property name="link_2_length" value="0.432" />
     <xacro:property name="link_2_radius" value="0.065278" />
     <joint name="joint_2" type="revolute">
@@ -95,7 +96,9 @@
         <dynamics damping="1.0" friction="1.0"/>
     </joint>
+    <!-- MATLAB Link 2 = link_2 (m2=17.4 kg) -->
+    <!-- CoG2 = [0.068; 0.006; -0.016] w.r.t. link frame {2} -->
     <link name="link_2">
         <visual>
-            <origin xyz="${link_2_length/2 - 0.226} 0 0" rpy="0 ${pi/2} 0"/>
+            <origin xyz="${link_2_length/2} 0 0" rpy="0 ${pi/2} 0"/>
             <geometry>
                 <cylinder length="${link_2_length}" radius="${link_2_radius}" />
@@ -104,5 +107,5 @@
         </visual>
         <collision>
-            <origin xyz="${link_2_length/2 - 0.226} 0 0" rpy="0 ${pi/2} 0"/>
+            <origin xyz="${link_2_length/2} 0 0" rpy="0 ${pi/2} 0"/>
             <geometry>
                 <cylinder length="${link_2_length}" radius="${link_2_radius}" />
@@ -113,8 +116,8 @@
         </xacro:inertial_cylinder>
     </link>
-    <xacro:property name="link_3_length" value="${0.4318 + 0.13208}" />
+    <xacro:property name="link_3_length" value="0.233" />
     <xacro:property name="link_3_radius" value="0.028702" />
     <joint name="joint_3" type="revolute">
-        <origin xyz="${link_2_length - 0.226 - link_3_radius} -${link_2_radius + link_3_radius} 0" rpy="0 0 0"/>
+        <origin xyz="${link_2_length} -0.094 0" rpy="0 0 0"/>
         <parent link="link_2"/>
         <child link="link_3"/>
@@ -123,7 +126,9 @@
         <dynamics damping="1.0" friction="1.0"/>
     </joint>
+    <!-- MATLAB Link 3 = link_3 (m3=4.8 kg) -->
+    <!-- CoG3 = [0.000; -0.143; 0.014] w.r.t. link frame {3} -->
     <link name="link_3">
         <visual>
-            <origin xyz="0 0 ${link_3_length/2 - 0.4318}" rpy="0 0 0"/>
+            <origin xyz="0 0 -${link_3_length/2}" rpy="0 0 0"/>
             <geometry>
                 <cylinder length="${link_3_length}" radius="${link_3_radius}" />
@@ -132,5 +137,5 @@
         </visual>
         <collision>
-            <origin xyz="0 0 ${link_3_length/2 - 0.4318}" rpy="0 0 0"/>
+            <origin xyz="0 0 -${link_3_length/2}" rpy="0 0 0"/>
             <geometry>
                 <cylinder length="${link_3_length}" radius="${link_3_radius}" />

Commit message: kadasi update

File: arm_bot/src/description/robot_core.xacro (robot description, xacro)
@@ -92,5 +92,5 @@
         <parent link="shoulder"/>
         <child link="link_2"/>
-        <axis xyz="0 -1 0"/>
+        <axis xyz="0 1 0"/>
         <limit lower="-1" upper="3.363" velocity="1" effort="100"/>
         <dynamics damping="1.0" friction="1.0"/>
@@ -122,5 +122,5 @@
         <parent link="link_2"/>
         <child link="link_3"/>
-        <axis xyz="0 -1 0"/>
+        <axis xyz="0 1 0"/>
         <limit lower="-0.712" upper="4" velocity="1" effort="100"/>
         <dynamics damping="1.0" friction="1.0"/>
@@ -130,5 +130,5 @@
     <link name="link_3">
         <visual>
-            <origin xyz="0 0 -${link_3_length/2}" rpy="0 0 0"/>
+            <origin xyz="0 0 ${link_3_length/2}" rpy="0 0 0"/>
             <geometry>
                 <cylinder length="${link_3_length}" radius="${link_3_radius}" />

Commit message: finetuning

File: arm_bot/src/description/robot_core.xacro (robot description, xacro)
@@ -65,5 +65,5 @@
         <axis xyz="0 0 1"/>
         <limit lower="0" upper="5.585" velocity="1" effort="100"/>
-        <dynamics damping="1.0" friction="1.0"/>
+        <dynamics damping="0" friction="0"/>
     </joint>
     <!-- MATLAB Link 1 = shoulder (m1=0, only Izz=1.49) -->
@@ -94,5 +94,5 @@
         <axis xyz="0 1 0"/>
         <limit lower="-1" upper="3.363" velocity="1" effort="100"/>
-        <dynamics damping="1.0" friction="1.0"/>
+        <dynamics damping="0" friction="0"/>
     </joint>
     <!-- MATLAB Link 2 = link_2 (m2=17.4 kg) -->
@@ -124,5 +124,5 @@
         <axis xyz="0 1 0"/>
         <limit lower="-0.712" upper="4" velocity="1" effort="100"/>
-        <dynamics damping="1.0" friction="1.0"/>
+        <dynamics damping="0" friction="0"/>
     </joint>
     <!-- MATLAB Link 3 = link_3 (m3=4.8 kg) -->

Commit message: model and script update

File: arm_bot/src/description/robot_core.xacro (robot description, xacro)
@@ -41,6 +41,8 @@
         <visual>
             <origin xyz="0 0 ${link_1_length/2}" rpy="0 0 0"/>
+            <!-- <origin xyz="0 0 0" rpy="0 0 ${pi/2}"/> -->
             <geometry>
                 <cylinder length="${link_1_length}" radius="${link_1_radius}" />
+                 <!-- <mesh filename="package://arm_bot/meshes/puma_link1.stl" scale="0.0254 0.0254 0.0254"/> -->
             </geometry>
             <material name="blue" />
@@ -50,4 +52,5 @@
             <geometry>
                 <cylinder length="${link_1_length}" radius="${link_1_radius}" />
+                 <!-- <mesh filename="package://arm_bot/meshes/puma_link1.stl" scale="0.0254 0.0254 0.0254"/> -->
             </geometry>
         </collision>
@@ -64,5 +67,5 @@
         <child link="shoulder"/>
         <axis xyz="0 0 1"/>
-        <limit lower="0" upper="5.585" velocity="1" effort="100"/>
+        <limit lower="${-8*pi/9}" upper="${8*pi/9}" velocity="2" effort="1000"/>
         <dynamics damping="0" friction="0"/>
     </joint>
@@ -71,6 +74,8 @@
         <visual>
             <origin xyz="0 ${shoulder_length/2 - shoulder_radius} 0" rpy="${pi/2} 0 0"/>
+            <!-- <origin xyz="0 -0.09677 0" rpy="${pi/2} 0 ${pi}"/> -->
             <geometry>
                 <cylinder length="${shoulder_length}" radius="${shoulder_radius}" />
+                 <!-- <mesh filename="package://arm_bot/meshes/puma_link2.stl" scale="0.0254 0.0254 0.0254"/> -->
             </geometry>
             <material name="blue" />
@@ -89,9 +94,9 @@
     <xacro:property name="link_2_radius" value="0.065278" />
     <joint name="joint_2" type="revolute">
-        <origin xyz="0 ${shoulder_length} 0" rpy="0 0 0"/>
+        <origin xyz="0 ${shoulder_length} 0" rpy="${-pi/2} 0 0"/>
         <parent link="shoulder"/>
         <child link="link_2"/>
-        <axis xyz="0 1 0"/>
-        <limit lower="-1" upper="3.363" velocity="1" effort="100"/>
+        <axis xyz="0 0 1"/>
+        <limit lower="${-5*pi/4}" upper="${pi/4}" velocity="2" effort="1000"/>
         <dynamics damping="0" friction="0"/>
     </joint>
@@ -101,6 +106,8 @@
         <visual>
             <origin xyz="${link_2_length/2} 0 0" rpy="0 ${pi/2} 0"/>
+            <!-- <origin xyz="0 0 0" rpy="${3*pi/2} 0 0"/> -->
             <geometry>
                 <cylinder length="${link_2_length}" radius="${link_2_radius}" />
+                 <!-- <mesh filename="package://arm_bot/meshes/puma_link3.stl" scale="0.0254 0.0254 0.0254"/> -->
             </geometry>
             <material name="orange" />
@@ -119,9 +126,9 @@
     <xacro:property name="link_3_radius" value="0.028702" />
     <joint name="joint_3" type="revolute">
-        <origin xyz="${link_2_length} -0.094 0" rpy="0 0 0"/>
+        <origin xyz="${link_2_length} 0 -0.094" rpy="0 0 0"/>
         <parent link="link_2"/>
         <child link="link_3"/>
-        <axis xyz="0 1 0"/>
-        <limit lower="-0.712" upper="4" velocity="1" effort="100"/>
+        <axis xyz="0 0 1"/>
+        <limit lower="${-pi/4}" upper="${5*pi/4}" velocity="2" effort="1000"/>
         <dynamics damping="0" friction="0"/>
     </joint>
@@ -130,12 +137,14 @@
     <link name="link_3">
         <visual>
-            <origin xyz="0 0 ${link_3_length/2}" rpy="0 0 0"/>
+            <origin xyz="0 -${link_3_length/2} 0" rpy="${-pi/2} 0 0"/>
+            <!-- <origin xyz="0 ${0.094/2} 0" rpy="${pi/2} -${pi/2} 0"/> -->
             <geometry>
                 <cylinder length="${link_3_length}" radius="${link_3_radius}" />
+                 <!-- <mesh filename="package://arm_bot/meshes/puma_link4.stl" scale="0.0254 0.0254 0.0254"/> -->
             </geometry>
             <material name="yellow" />
         </visual>
         <collision>
-            <origin xyz="0 0 -${link_3_length/2}" rpy="0 0 0"/>
+            <origin xyz="0 -${link_3_length/2} 0" rpy="${-pi/2} 0 0"/>
             <geometry>
                 <cylinder length="${link_3_length}" radius="${link_3_radius}" />

Commit message: collision update for robot and script update

File: arm_bot/src/description/robot_core.xacro (robot description, xacro)
@@ -49,8 +49,9 @@
         </visual>
         <collision>
-            <origin xyz="0 0 ${link_1_length/2}" rpy="0 0 0"/>
+            <!-- <origin xyz="0 0 ${link_1_length/2}" rpy="0 0 0"/> -->
+            <origin xyz="0 0 0" rpy="0 0 ${-pi/2}"/>
             <geometry>
-                <cylinder length="${link_1_length}" radius="${link_1_radius}" />
-                 <!-- <mesh filename="package://arm_bot/meshes/puma_link1.stl" scale="0.0254 0.0254 0.0254"/> -->
+                <!-- <cylinder length="${link_1_length}" radius="${link_1_radius}" /> -->
+                 <mesh filename="package://arm_bot/meshes/puma_link1.stl" scale="0.0254 0.0254 0.0254"/>
             </geometry>
         </collision>
@@ -82,7 +83,9 @@
         </visual>
         <collision>
-            <origin xyz="0 ${shoulder_length/2 - shoulder_radius} 0" rpy="${pi/2} 0 0"/>
+            <!-- <origin xyz="0 ${shoulder_length/2 - shoulder_radius} 0" rpy="${pi/2} 0 0"/> -->
+            <origin xyz="0 -0.09677 0" rpy="${pi/2} 0 ${pi}"/>
             <geometry>
-                <cylinder length="${shoulder_length}" radius="${shoulder_radius}" />
+                <!-- <cylinder length="${shoulder_length}" radius="${shoulder_radius}" /> -->
+                 <mesh filename="package://arm_bot/meshes/puma_link2.stl" scale="0.0254 0.0254 0.0254"/>
             </geometry>
         </collision>
@@ -114,7 +117,9 @@
         </visual>
         <collision>
-            <origin xyz="${link_2_length/2} 0 0" rpy="0 ${pi/2} 0"/>
+            <!-- <origin xyz="${link_2_length/2} 0 0" rpy="0 ${pi/2} 0"/> -->
+            <origin xyz="0 0 0" rpy="0 0 0"/>
             <geometry>
-                <cylinder length="${link_2_length}" radius="${link_2_radius}" />
+                <!-- <cylinder length="${link_2_length}" radius="${link_2_radius}" /> -->
+                 <mesh filename="package://arm_bot/meshes/puma_link3.stl" scale="0.0254 0.0254 0.0254"/>
             </geometry>
         </collision>
@@ -146,7 +151,9 @@
         </visual>
         <collision>
-            <origin xyz="0 -${link_3_length/2} 0" rpy="${-pi/2} 0 0"/>
+            <!-- <origin xyz="0 -${link_3_length/2} 0" rpy="${-pi/2} 0 0"/> -->
+            <origin xyz="0 0 ${0.094/2}" rpy="0 0 ${-pi/2}"/>
             <geometry>
-                <cylinder length="${link_3_length}" radius="${link_3_radius}" />
+                <!-- <cylinder length="${link_3_length}" radius="${link_3_radius}" /> -->
+                 <mesh filename="package://arm_bot/meshes/puma_link4.stl" scale="0.0254 0.0254 0.0254"/>
             </geometry>
         </collision>
