Commit message: update_3
Co-authored-by: Copilot <copilot@github.com>

File: arm_bot/src/description/robot_core.xacro (robot description, xacro)
@@ -101,6 +101,6 @@
         <child link="link_2"/>
         <axis xyz="0 0 1"/>
-        <limit lower="${-5*pi/4}" upper="${pi/4}" velocity="2" effort="1000"/>
-        <dynamics damping="0" friction="0"/>
+        <limit lower="${-5*pi/4}" upper="${pi/3}" velocity="2" effort="1000"/>
+        <dynamics damping="1" friction="0"/>
     </joint>
     <!-- MATLAB Link 2 = link_2 (m2=17.4 kg) -->
@@ -136,5 +136,5 @@
         <axis xyz="0 0 1"/>
         <limit lower="${-pi/4}" upper="${5*pi/4}" velocity="2" effort="1000"/>
-        <dynamics damping="0" friction="0"/>
+        <dynamics damping="1" friction="0"/>
     </joint>
     <!-- MATLAB Link 3 = link_3 (m3=4.8 kg) -->
@@ -146,5 +146,5 @@
             <geometry>
                 <!-- <cylinder length="${link_3_length}" radius="${link_3_radius}" /> -->
-                 <mesh filename="package://arm_bot/meshes/puma_link4.stl" scale="0.0254 0.0254 0.0254"/>
+                 <mesh filename="package://arm_bot/meshes/puma_link4.stl" scale="0.02 0.02 0.02"/>
             </geometry>
             <material name="yellow" />
@@ -155,5 +155,5 @@
             <geometry>
                 <!-- <cylinder length="${link_3_length}" radius="${link_3_radius}" /> -->
-                 <mesh filename="package://arm_bot/meshes/puma_link4.stl" scale="0.0254 0.0254 0.0254"/>
+                 <mesh filename="package://arm_bot/meshes/puma_link4.stl" scale="0.02 0.02 0.02"/>
             </geometry>
         </collision>

File: arm_bot/src/description/ros2_control.xacro (robot description, xacro)
@@ -16,5 +16,7 @@
                     <param name="initial_value">0</param>
                 </state_interface>
-                <state_interface name="effort"/>
+                <state_interface name="effort">
+                    <param name="initial_value">${0.0}</param>
+                </state_interface>
             </joint>
             <joint name="joint_2">
@@ -27,5 +29,7 @@
                     <param name="initial_value">${pi/4}</param>
                 </state_interface>
-                <state_interface name="effort"/>
+                <state_interface name="effort">
+                    <param name="initial_value">${-21.83836502601828}</param>
+                </state_interface>
             </joint>
             <joint name="joint_3">
@@ -38,5 +42,7 @@
                     <param name="initial_value">${3*pi/4}</param>
                 </state_interface>
-                <state_interface name="effort"/>
+                <state_interface name="effort">
+                    <param name="initial_value">${0.0}</param>
+                </state_interface>
             </joint>
         </ros2_control>

Commit message: improved_1
Co-authored-by: Copilot <copilot@github.com>

File: arm_bot/src/description/robot_core.xacro (robot description, xacro)
@@ -102,5 +102,5 @@
         <axis xyz="0 0 1"/>
         <limit lower="${-5*pi/4}" upper="${pi/3}" velocity="2" effort="1000"/>
-        <dynamics damping="1" friction="0"/>
+        <dynamics damping="0.5" friction="0"/>
     </joint>
     <!-- MATLAB Link 2 = link_2 (m2=17.4 kg) -->
@@ -136,5 +136,5 @@
         <axis xyz="0 0 1"/>
         <limit lower="${-pi/4}" upper="${5*pi/4}" velocity="2" effort="1000"/>
-        <dynamics damping="1" friction="0"/>
+        <dynamics damping="0.5" friction="0"/>
     </joint>
     <!-- MATLAB Link 3 = link_3 (m3=4.8 kg) -->
