Commit message: pos controller update

File: arm_bot_pos_control/src/description/robot_core.xacro (robot description, xacro)
@@ -44,13 +44,14 @@
             <geometry>
                 <!-- <cylinder length="${link_1_length}" radius="${link_1_radius}" /> -->
-                 <mesh filename="package://arm_bot/meshes/puma_link1.stl" scale="0.0254 0.0254 0.0254"/>
+                 <mesh filename="package://arm_bot_pos_control/meshes/puma_link1.stl" scale="0.0254 0.0254 0.0254"/>
             </geometry>
             <material name="purple" />
         </visual>
         <collision>
-            <origin xyz="0 0 ${link_1_length/2}" rpy="0 0 0"/>
+            <!-- <origin xyz="0 0 ${link_1_length/2}" rpy="0 0 0"/> -->
+            <origin xyz="0 0 0" rpy="0 0 ${-pi/2}"/>
             <geometry>
-                <cylinder length="${link_1_length}" radius="${link_1_radius}" />
-                 <!-- <mesh filename="package://arm_bot/meshes/puma_link1.stl" scale="0.0254 0.0254 0.0254"/> -->
+                <!-- <cylinder length="${link_1_length}" radius="${link_1_radius}" /> -->
+                 <mesh filename="package://arm_bot_pos_control/meshes/puma_link1.stl" scale="0.0254 0.0254 0.0254"/>
             </geometry>
         </collision>
@@ -77,12 +78,14 @@
             <geometry>
                 <!-- <cylinder length="${shoulder_length}" radius="${shoulder_radius}" /> -->
-                 <mesh filename="package://arm_bot/meshes/puma_link2.stl" scale="0.0254 0.0254 0.0254"/>
+                 <mesh filename="package://arm_bot_pos_control/meshes/puma_link2.stl" scale="0.0254 0.0254 0.0254"/>
             </geometry>
             <material name="blue" />
         </visual>
         <collision>
-            <origin xyz="0 ${shoulder_length/2 - shoulder_radius} 0" rpy="${pi/2} 0 0"/>
+            <!-- <origin xyz="0 ${shoulder_length/2 - shoulder_radius} 0" rpy="${pi/2} 0 0"/> -->
+            <origin xyz="0 -0.09677 0" rpy="${pi/2} 0 ${pi}"/>
             <geometry>
-                <cylinder length="${shoulder_length}" radius="${shoulder_radius}" />
+                <!-- <cylinder length="${shoulder_length}" radius="${shoulder_radius}" /> -->
+                 <mesh filename="package://arm_bot_pos_control/meshes/puma_link2.stl" scale="0.0254 0.0254 0.0254"/>
             </geometry>
         </collision>
@@ -109,12 +112,14 @@
             <geometry>
                 <!-- <cylinder length="${link_2_length}" radius="${link_2_radius}" /> -->
-                 <mesh filename="package://arm_bot/meshes/puma_link3.stl" scale="0.0254 0.0254 0.0254"/>
+                 <mesh filename="package://arm_bot_pos_control/meshes/puma_link3.stl" scale="0.0254 0.0254 0.0254"/>
             </geometry>
             <material name="orange" />
         </visual>
         <collision>
-            <origin xyz="${link_2_length/2} 0 0" rpy="0 ${pi/2} 0"/>
+            <!-- <origin xyz="${link_2_length/2} 0 0" rpy="0 ${pi/2} 0"/> -->
+            <origin xyz="0 0 0" rpy="0 0 0"/>
             <geometry>
-                <cylinder length="${link_2_length}" radius="${link_2_radius}" />
+                <!-- <cylinder length="${link_2_length}" radius="${link_2_radius}" /> -->
+                 <mesh filename="package://arm_bot_pos_control/meshes/puma_link3.stl" scale="0.0254 0.0254 0.0254"/>
             </geometry>
         </collision>
@@ -141,12 +146,14 @@
             <geometry>
                 <!-- <cylinder length="${link_3_length}" radius="${link_3_radius}" /> -->
-                 <mesh filename="package://arm_bot/meshes/puma_link4.stl" scale="0.0254 0.0254 0.0254"/>
+                 <mesh filename="package://arm_bot_pos_control/meshes/puma_link4.stl" scale="0.0254 0.0254 0.0254"/>
             </geometry>
             <material name="yellow" />
         </visual>
         <collision>
-            <origin xyz="0 -${link_3_length/2} 0" rpy="${-pi/2} 0 0"/>
+            <!-- <origin xyz="0 -${link_3_length/2} 0" rpy="${-pi/2} 0 0"/> -->
+            <origin xyz="0 0 ${0.094/2}" rpy="0 0 ${-pi/2}"/>
             <geometry>
-                <cylinder length="${link_3_length}" radius="${link_3_radius}" />
+                <!-- <cylinder length="${link_3_length}" radius="${link_3_radius}" /> -->
+                 <mesh filename="package://arm_bot_pos_control/meshes/puma_link4.stl" scale="0.0254 0.0254 0.0254"/>
             </geometry>
         </collision>

File: arm_bot_pos_control/src/description/ros2_control.xacro (robot description, xacro)
@@ -10,5 +10,7 @@
                 <command_interface name="position"/>
                 <state_interface name="velocity"/>
-                <state_interface name="position"/>
+                <state_interface name="position">
+                    <param name="initial_value">0</param>
+                </state_interface>
                 <state_interface name="effort"/>
             </joint>
@@ -16,5 +18,7 @@
                 <command_interface name="position"/>
                 <state_interface name="velocity"/>
-                <state_interface name="position"/>
+                <state_interface name="position">
+                    <param name="initial_value">${0}</param>
+                </state_interface>
                 <state_interface name="effort"/>
             </joint>
@@ -22,5 +26,7 @@
                 <command_interface name="position"/>
                 <state_interface name="velocity"/>
-                <state_interface name="position"/>
+                <state_interface name="position">
+                    <param name="initial_value">${3*pi/4}</param>
+                </state_interface>
                 <state_interface name="effort"/>
             </joint>

Commit message: position controler update

File: arm_bot_pos_control/src/description/robot_core.xacro (robot description, xacro)
@@ -101,5 +101,5 @@
         <child link="link_2"/>
         <axis xyz="0 0 1"/>
-        <limit lower="${-5*pi/4}" upper="${pi/4}" velocity="2" effort="1000"/>
+        <limit lower="${-5*pi/4}" upper="${pi/2}" velocity="2" effort="1000"/>
         <dynamics damping="0" friction="0"/>
     </joint>

File: arm_bot_pos_control/src/description/ros2_control.xacro (robot description, xacro)
@@ -19,5 +19,5 @@
                 <state_interface name="velocity"/>
                 <state_interface name="position">
-                    <param name="initial_value">${0}</param>
+                    <param name="initial_value">${pi/4}</param>
                 </state_interface>
                 <state_interface name="effort"/>

Commit message: added friction

File: arm_bot_pos_control/src/description/robot_core.xacro (robot description, xacro)
@@ -69,5 +69,5 @@
         <axis xyz="0 0 1"/>
         <limit lower="${-8*pi/9}" upper="${8*pi/9}" velocity="2" effort="1000"/>
-        <dynamics damping="0" friction="0"/>
+        <dynamics damping="4" friction="3"/>
     </joint>
     <!-- MATLAB Link 1 = shoulder (m1=0, only Izz=1.49) -->
@@ -102,5 +102,5 @@
         <axis xyz="0 0 1"/>
         <limit lower="${-5*pi/4}" upper="${pi/2}" velocity="2" effort="1000"/>
-        <dynamics damping="0" friction="0"/>
+        <dynamics damping="5" friction="5"/>
     </joint>
     <!-- MATLAB Link 2 = link_2 (m2=17.4 kg) -->
@@ -136,5 +136,5 @@
         <axis xyz="0 0 1"/>
         <limit lower="${-pi/4}" upper="${5*pi/4}" velocity="2" effort="1000"/>
-        <dynamics damping="0" friction="0"/>
+        <dynamics damping="4" friction="5"/>
     </joint>
     <!-- MATLAB Link 3 = link_3 (m3=4.8 kg) -->
